Commit message: basic URDF finished

File: electric_jacker_description/urdf/robot.urdf (robot description, URDF)
Before this commit: robot electric_jacker, 6 links, 5 joints
Links:
- added link left_fork_caster_link, mass 0.5; collision sphere radius=0.025; visual sphere radius=0.025
Joints:
- added joint left_fork_caster_joint: type fixed, parent left_fork_link, child left_fork_caster_link, origin xyz=0.0762 1 0 rpy=-1.57079632679 0 0
- joint right_fork_caster_joint: origin xyz=0.115 0.0 0.007 rpy=-1.57079632679 0 0 -> xyz=0.0762 1 0 rpy=-1.57079632679 0 0

Commit message: gazebo running

File: electric_jacker_description/urdf/robot.urdf (robot description, URDF)
Before this commit: robot electric_jacker, 7 links, 6 joints
Links:
- link base_link: mass None -> 22
- link left_fork_link: mass None -> 22

Commit message: Gazebo and Twist Teleop Work

File: electric_jacker_description/urdf/robot.urdf (robot description, URDF)
Before this commit: robot electric_jacker, 7 links, 6 joints
Joints:
- joint left_fork_joint: origin xyz=.19 .12 0 rpy=0 0 0 -> xyz=.19 .12 0.025 rpy=0 0 0
- joint left_wheel_joint: origin xyz=-0.27 0 0.065 rpy=0 0 0 -> xyz=-0.27 0 0.09 rpy=0 0 0
- joint right_fork_joint: origin xyz=-.34 .12 0 rpy=0 0 0 -> xyz=-.34 .12 0.025 rpy=0 0 0
- joint right_wheel_joint: origin xyz=0.27 0 0.065 rpy=0 0 0 -> xyz=0.27 0 0.09 rpy=0 0 0

Commit message: Complete Success in Gazebo

File: electric_jacker_description/urdf/robot.urdf (robot description, URDF)
Before this commit: robot electric_jacker, 7 links, 6 joints
Links:
- added link base_footprint; visual box size=0.001 0.001 0.001
- link base_link: mass 22 -> 15
- link left_fork_link: mass 22 -> 10
- link right_fork_link: mass None -> 10
Joints:
- added joint base_footprint_joint: type fixed, parent base_footprint, child base_link, origin xyz=0 0 0.04 rpy=0 0 0

Commit message: added camera to robot

File: electric_jacker_description/urdf/robot.urdf (robot description, URDF)
Before this commit: robot electric_jacker, 8 links, 7 joints
Links:
- added link camera_depth_frame, mass 0.001
- added link camera_depth_optical_frame, mass 0.001
- added link camera_link, mass 0.001; collision box size=0.07271 0.27794 0.073; visual mesh filename=package://electric_jacker_description/models/meshes/kinect.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
- added link camera_rgb_frame, mass 0.001
- added link camera_rgb_optical_frame, mass 0.001
Joints:
- added joint camera_depth_joint: type fixed, parent camera_rgb_frame, child camera_depth_frame, origin xyz=0 0.0 0 rpy=0 0 0
- added joint camera_depth_optical_joint: type fixed, parent camera_depth_frame, child camera_depth_optical_frame, origin xyz=0 0 0 rpy=-1.57079632679 0 -1.57079632679
- added joint camera_joint: type fixed, parent camera_rgb_frame, child camera_link, origin xyz=-0.031 -0.0 -0.016 rpy=0 0 0
- added joint camera_rgb_joint: type fixed, parent base_link, child camera_rgb_frame, origin xyz=0.0 -0.127 0.1778 rpy=0 0 0
- added joint camera_rgb_optical_joint: type fixed, parent camera_rgb_frame, child camera_rgb_optical_frame, origin xyz=0 0 0 rpy=-1.57079632679 0 -1.57079632679
- joint left_wheel_joint: axis -1 0 0 -> 1 0 0
- joint right_wheel_joint: axis -1 0 0 -> 1 0 0
